Commit message: Modified jackal_description for docking: docking_fixture, tag36_11_00002

File: jackal_description/urdf/accessories.urdf.xacro (robot description, xacro)
@@ -461,3 +461,31 @@
     </gazebo>
   </xacro:if>
+  <!-- Docking fixture (enable with JACKAL_DOCKING=1 in configs/docking) -->
+  <xacro:include filename="$(find jackal_description)/urdf/accessories/docking_fixture.urdf.xacro" />
+  <xacro:if value="$(optenv JACKAL_DOCKING 0)">
+    <xacro:property name="parent"       value="$(optenv JACKAL_DOCKINGFIXTURE_PARENT mid_mount)" />
+    <xacro:property name="fixture_xyz"  value="$(optenv JACKAL_DOCKINGFIXTURE_OFFSET 0 0 0.12)" />
+    <xacro:property name="fixture_rpy"  value="$(optenv JACKAL_DOCKINGFIXTURE_RPY 0 0 0)" />
+    <xacro:property name="mesh"         value="$(optenv JACKAL_DOCKINGFIXTURE_MESH package://jackal_description/meshes/docking_fixture.dae)" />
+    <xacro:property name="scale"        value="$(optenv JACKAL_DOCKINGFIXTURE_SCALE 1 1 1)" />
+    <xacro:property name="mass"         value="$(optenv JACKAL_DOCKINGFIXTURE_MASS 1.0)" />
+    <xacro:docking_fixture   parent_link ="${parent}"
+                             mesh_file   ="${mesh}"
+                             scale       ="${scale}"
+                             mass        ="${mass}"
+                             fixture_xyz ="${fixture_xyz}" fixture_rpy ="${fixture_rpy}" />
+  </xacro:if>
+  <!-- AprilTag accessory (enable with JACKAL_TAG=1 in configs/docking) -->
+  <xacro:include filename="$(find jackal_description)/urdf/accessories/apriltag.urdf.xacro"/>
+  <xacro:if value="$(optenv JACKAL_TAG 0)">
+    <xacro:property name="dock_xyz"     value="$(optenv JACKAL_DOCK_XYZ 0 0 0)" />
+    <xacro:property name="dock_rpy"     value="$(optenv JACKAL_DOCK_RPY 0 0 0)" />
+    <xacro:apriltag         parent_link ="$(optenv JACKAL_TAG_PARENT mid_mount)"
+                            size        ="$(optenv JACKAL_TAG_SIZE 1.0)"
+                            thickness   ="$(optenv JACKAL_TAG_THICKNESS 0.003)"
+                            mesh_file   ="$(optenv JACKAL_TAG_MESH package://jackal_description/meshes/tag36_11_00002.dae)"
+                            tag_xyz         ="$(optenv JACKAL_TAG_OFFSET 0 0 0)"
+                            tag_rpy         ="$(optenv JACKAL_TAG_RPY 0 0 0)"
+                            dock_xyz    ="${dock_xyz}"  dock_rpy="${dock_rpy}" />
+  </xacro:if>
 </robot>

Commit message: fix apriltag_frame, dock pose (xyz, rpy), fixture/dock collisions, docking config file

File: jackal_description/urdf/accessories.urdf.xacro (robot description, xacro)
@@ -465,5 +465,5 @@
   <xacro:if value="$(optenv JACKAL_DOCKING 0)">
     <xacro:property name="parent"       value="$(optenv JACKAL_DOCKINGFIXTURE_PARENT mid_mount)" />
-    <xacro:property name="fixture_xyz"  value="$(optenv JACKAL_DOCKINGFIXTURE_OFFSET 0 0 0.12)" />
+    <xacro:property name="fixture_xyz"  value="$(optenv JACKAL_DOCKINGFIXTURE_OFFSET 0 0 0.12)" />  <!-- 0 0 0.12 -->
     <xacro:property name="fixture_rpy"  value="$(optenv JACKAL_DOCKINGFIXTURE_RPY 0 0 0)" />
     <xacro:property name="mesh"         value="$(optenv JACKAL_DOCKINGFIXTURE_MESH package://jackal_description/meshes/docking_fixture.dae)" />
@@ -485,7 +485,8 @@
                             thickness   ="$(optenv JACKAL_TAG_THICKNESS 0.003)"
                             mesh_file   ="$(optenv JACKAL_TAG_MESH package://jackal_description/meshes/tag36_11_00002.dae)"
-                            tag_xyz         ="$(optenv JACKAL_TAG_OFFSET 0 0 0)"
-                            tag_rpy         ="$(optenv JACKAL_TAG_RPY 0 0 0)"
-                            dock_xyz    ="${dock_xyz}"  dock_rpy="${dock_rpy}" />
+                            tag_xyz     ="$(optenv JACKAL_TAG_OFFSET 0 0 0)"
+                            tag_rpy     ="$(optenv JACKAL_TAG_RPY 0 0 0)"
+                            dock_xyz    ="${dock_xyz}"
+                            dock_rpy    ="${dock_rpy}" />
   </xacro:if>
 </robot>

File: jackal_description/urdf/accessories/apriltag.urdf.xacro (robot description, xacro)
@@ -11,5 +11,5 @@
                        density:=900.0
                        dock_xyz:= '0 0 0'
-                       dock_rpy:= '0 0 0'">    <!-- kg/m^3: light plastic/foam-ish -->
+                       dock_rpy:= '0 0 0'">    <!-- kg/m³: light plastic/foam-ish (0.9 g/cm³)-->
     <xacro:property name="mass" value="${size*size*thickness*density}"/>
     <link name="apriltag_link">
@@ -24,5 +24,4 @@
                  ixy="0" ixz="0" iyz="0"/>
       </inertial>
-      <!-- Visual: DO NOT add a <material> here; let the DAE texture show -->
       <visual>
         <origin xyz="0 0 0" rpy="0 0 0"/>
@@ -45,7 +44,7 @@
       <origin xyz="${tag_xyz}" rpy="${tag_rpy}"/>
     </joint>
-    <gazebo reference="apriltag_link">
+    <!-- <gazebo reference="apriltag_link">
       <turnGravityOff>false</turnGravityOff>
-      <!-- <material>
+      <!- - <material>
         <script> <!- - one more way to make it brighter - use .sdf files settings, try if necessary, og - ->
           <uri>model://Apriltag36_11_00002/materials/scripts</uri>
@@ -53,8 +52,16 @@
           <name>Apriltag36_11_00002</name>
         </script>
-      </material> -->
-      <!-- <lighting>false</lighting> <!- - "" .... og - -> -->
-    </gazebo>
-    <link name="dock"/>
+      </material> - ->
+      <!- - <lighting>false</lighting> <!- - "" .... og - -> - ->
+    </gazebo>  -->
+    <link name="dock">
+      <collision>
+        <origin xyz="0.15 0 0" rpy="0 1.5708 0"/>
+        <geometry>
+          <cylinder radius="0.02" length="0.1" />
+          <!-- <mesh filename="${mesh_file}" scale="${scale}"/> -->
+        </geometry>
+      </collision>
+    </link>
     <joint name="dock_joint" type="fixed">
       <parent link="apriltag_link"/>

File: jackal_description/urdf/accessories/docking_fixture.urdf.xacro (robot description, xacro)
@@ -28,11 +28,9 @@
         <!-- <material name="dark_grey"/> -->
       </visual>
-      <!-- Keep collision simple at first for stability; swap to mesh if needed -->
       <collision>
-        <origin xyz="0 0 0" rpy="0 0 0"/>
+        <origin xyz="0.09 0 0.25" rpy="0 0 0"/>
         <geometry>
-          <!-- Approximate as a box initially; replace with mesh if needed -->
-          <!-- <box size="0.200 0.315 0.500"/> -->
-          <mesh filename="${mesh_file}" scale="${scale}"/>
+          <box size="0.200 0.315 0.500"/>
+          <!-- <mesh filename="${mesh_file}" scale="${scale}"/> -->
         </geometry>
       </collision>
